Commit message: 20/03/22

File: src/tx2_slam/urdf/zed_descr.urdf.xacro (robot description, xacro)
@@ -19,7 +19,7 @@
     <xacro:include filename="$(find zed_wrapper)/urdf/include/materials.urdf.xacro" />
     <!-- Arguments -->
-    <xacro:arg name="camera_name"   default="zed2" />
+    <xacro:arg name="camera_name"   default="tx2zed2" />
     <xacro:arg name="camera_model"  default="zed2" />
-    <xacro:arg name="base_frame"    default="base_link" />
+    <xacro:arg name="base_frame"    default="zed2_base_link" />
     <xacro:arg name="cam_pos_x"     default="0.0" />
     <xacro:arg name="cam_pos_y"     default="0.0" />
@@ -52,5 +52,5 @@
             <origin xyz="0 0 0" rpy="0 0 0"/>
             <geometry>
-                <mesh filename="package://zed_wrapper/urdf/models/${model}.stl" />
+                <mesh filename="package://tx2_slam/urdf/models/${model}.stl" />
             </geometry>
             <material name="${model}_mat" />
