Commit message: develope UI and add car model in urdf

File: src/tx2_slam/urdf/include/materials.urdf.xacro (robot description, xacro)
@@ -23,5 +23,5 @@
     </material>
     <material name="zed2_mat">
-        <color rgba="1 0.25 0.25 0.99"/>
+        <color rgba="1 0.89 0.07 1"/>
     </material>
 </robot>

File: src/tx2_slam/urdf/zed_descr.urdf.xacro (robot description, xacro)
@@ -17,5 +17,5 @@
 <robot name="stereolabs_camera" xmlns:xacro="http://ros.org/wiki/xacro">
 <!-- Includes -->
-    <xacro:include filename="$(find zed_wrapper)/urdf/include/materials.urdf.xacro" />
+    <xacro:include filename="$(find tx2_slam)/urdf/include/materials.urdf.xacro" />
     <!-- Arguments -->
     <xacro:arg name="camera_name"   default="tx2zed2" />
@@ -50,7 +50,7 @@
     <link name="$(arg camera_name)_camera_center">
         <visual>
-            <origin xyz="0 0 0" rpy="0 0 0"/>
+            <origin xyz="0 0 0" rpy="1.57 0 0"/>
             <geometry>
-                <mesh filename="package://tx2_slam/urdf/models/${model}.stl" />
+                <mesh filename="package://tx2_slam/urdf/models/robot_asm.stl" />
             </geometry>
             <material name="${model}_mat" />
